File: mmeshtastic-pcb.kicad_pcb (KiCad board)
At the start: 2 copper layers, 90.2 x 44.5 mm, 29 parts, among them J1 Conn_01x05, J2 Conn_01x02, M1 RP2040-LoRa-HF, Q1 FS8205A, U1 DW01A, U2 TP5000_Breakout_Akaddy, U3 LM2596 Module

Commit message: Run DRC, everything checks out
Other:
- board text added: "V1.0 https://github.com/Bir-Paragliding-Community/RP2040-Solar-PCB"
